File: hardware/AVR-Timer_smd.brd (EAGLE design)
At the start: 72.7 x 57.1 mm, 44 parts, among them IC1 MEGA8-AI, Q1 IRLML5203, Q2 IRLML5203, Q3 IRLML5203, Q4 IRLML5203, Q5 IRLML5203, X1 22-23-2021, X2 22-23-2021

Commit message: add Makefile and some notes to eagle files
Connections:
- net N$2 renamed RESET
