File: hardware/AVR-Timer_smd.sch (EAGLE design)
At the start: 44 parts, among them IC1 MEGA8-AI, Q1 IRLML5203, Q2 IRLML5203, Q3 IRLML5203, Q4 IRLML5203, Q5 IRLML5203, X1 22-23-2021, X2 22-23-2021

Commit message: add Makefile and some notes to eagle files
Connections:
- net N$2 renamed RESET
Changed lines of the file:
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@@
 <?xml version="1.0" encoding="utf-8"?>
 <!DOCTYPE eagle SYSTEM "eagle.dtd">
-<eagle version="6.1">
+<eagle version="7.4.0">
 <drawing>
 <settings>
@@
 </segment>
 </net>
-<net name="N$2" class="0">
+<net name="RESET" class="0">
 <segment>
 <pinref part="IC1" gate="G$1" pin="PC6(/RESET)"/>
